File: hardware/basicsensormodule.sch (KiCad schematic (older format))
At the start: 5 parts, among them U1 ZCS

Commit message: WARNING
Other:
- note added: "WARNING: PWM PIN NO CONECTED\n"
Changed lines of the file:
@@
 NoConn ~ 3000 5325
 NoConn ~ 3000 5375
+Text Notes 950  6350 0    394  ~ 79
+WARNING: PWM PIN NO CONECTED\n
 $EndSCHEMATC
